File: pcb/CANalog_nucleo.kicad_pcb (KiCad board)
At the start: 2 copper layers, 68.6 x 78.7 mm, 29 parts, among them J1 USB_B_Micro, J2 ENCODER, J3 AIN, J4 OLED, J5 AOUT, J6 DB9_Male, U1 NUCLEO64-F302R8, U2 ESP-01v090, U3 MCP6002-xSN, U4 SN65HVD230

Commit message: start new pcb layout
Parts:
- removed BT1: CR2032, Battery:BatteryHolder_Keystone_103_1x20mm
- removed G***: LOGO, PL_logo:logo_height_10mm
- removed J4: OLED, Connector_PinHeader_2.54mm:PinHeader_1x04_P2.54mm_Vertical
- added C10: 1uF, Capacitor_SMD:C_0805_2012Metric, F.Cu at (62.2, 40.9)
- added C11: 0.1uF, Capacitor_SMD:C_0805_2012Metric, F.Cu at (88.9, 83.5)
- added C4: 4.7uF, Capacitor_SMD:C_0805_2012Metric, F.Cu at (45.8, 148.2)
- added C5: 10uF, Capacitor_SMD:C_0805_2012Metric, F.Cu at (96.8, 29.4)
- added C6: 0.1uF, Capacitor_SMD:C_0805_2012Metric, F.Cu at (34.9, 147.8)
- added C7: 10uF, Capacitor_SMD:C_0805_2012Metric, F.Cu at (41.2, 141.9)
- added C8: 33pF, Capacitor_SMD:C_0603_1608Metric, F.Cu at (29.0, 149.9)
- added C9: 0.1uF, Capacitor_SMD:C_0805_2012Metric, F.Cu at (62.2, 43.9)
- added D1: LED, LED_SMD:LED_0603_1608Metric, F.Cu at (95.2, 37.4)
- added D10: LED, LED_SMD:LED_0603_1608Metric, F.Cu at (39.9, 98.5)
- added D2: SS14F, pl_Diode:SMAF, F.Cu at (164.6, 121.3)
- added D3: BZV55-C15, pl_Diode:Nexperia_BZV55_SOD80C, F.Cu at (69.0, 75.2)
- added D4: SS14F, pl_Diode:SMAF, F.Cu at (34.5, 141.2)
- added D5: 1N4148, Diode_THT:D_DO-35_SOD27_P7.62mm_Horizontal, F.Cu at (106.8, 26.4)
- added D6: SS14F, pl_Diode:SMAF, F.Cu at (25.5, 138.6)
- added D7: PESD1CAN-UX, Package_TO_SOT_SMD:SOT-323_SC-70, F.Cu at (82.4, 79.0)
- added D8: LED, LED_SMD:LED_0603_1608Metric, F.Cu at (39.7, 88.8)
- added D9: LED, LED_SMD:LED_0603_1608Metric, F.Cu at (39.5, 93.6)
- added JP2: TX_SELECT, Jumper:SolderJumper-3_P1.3mm_Bridged12_RoundedPad1.0x1.5mm, B.Cu at (112.7, 40.5)
- added JP3: RX_SELECT, Jumper:SolderJumper-3_P1.3mm_Bridged12_RoundedPad1.0x1.5mm, B.Cu at (112.7, 37.0)
- added JP4: BOOT0, Connector_PinHeader_2.54mm:PinHeader_1x02_P2.54mm_Vertical, F.Cu at (57.2, 58.5)
- added JP7: Jumper_3_Open, Connector_PinHeader_2.54mm:PinHeader_1x03_P2.54mm_Vertical, F.Cu at (61.2, 48.5)
- added JP8: Jumper_3_Open, Connector_PinHeader_2.54mm:PinHeader_1x03_P2.54mm_Vertical, F.Cu at (61.2, 34.0)
- added L1: 2.2uH, pl_Inductor:L_3.5mmx3.0mm_SMD, F.Cu at (23.3, 145.0)
- added Q1: DMP3099L-7, Package_TO_SOT_SMD:SOT-23, F.Cu at (64.1, 76.9)
- added Q2: MMBT2222A, Package_TO_SOT_SMD:SOT-23, F.Cu at (155.6, 121.2)
- added R14: 10k, Resistor_SMD:R_0805_2012Metric, F.Cu at (95.1, 35.1)
- added R15: 10k, Resistor_SMD:R_0805_2012Metric, F.Cu at (144.7, 120.2)
- added R16: 20k, Resistor_SMD:R_0805_2012Metric, F.Cu at (144.7, 124.1)
- added R17: 10k, Resistor_SMD:R_0805_2012Metric, F.Cu at (95.1, 32.6)
- added R18: 124k, Resistor_SMD:R_0805_2012Metric, F.Cu at (47.5, 141.5)
- added R19: 23.7k, Resistor_SMD:R_0805_2012Metric, F.Cu at (28.9, 144.7)
- added R20: 1k, Resistor_SMD:R_0805_2012Metric, F.Cu at (57.2, 63.2)
- added R21: 10k, Resistor_SMD:R_0805_2012Metric, F.Cu at (57.2, 67.7)
- added R22: 12k, Resistor_SMD:R_0805_2012Metric, F.Cu at (53.0, 45.4)
- added R23: 120k, Resistor_SMD:R_0805_2012Metric, F.Cu at (53.0, 42.4)
- added R24: 68k, Resistor_SMD:R_0805_2012Metric, F.Cu at (53.0, 39.5)
- added R25: 1k, Resistor_SMD:R_0805_2012Metric, F.Cu at (35.5, 93.7)
- added R26: 1k, Resistor_SMD:R_0805_2012Metric, F.Cu at (35.0, 88.8)
- added R27: 1k, Resistor_SMD:R_0805_2012Metric, F.Cu at (35.6, 98.4)
- added R28: 20k, Resistor_SMD:R_0805_2012Metric, F.Cu at (149.9, 120.2)
- added SW1: SW_Push, Button_Switch_THT:SW_PUSH_6mm, F.Cu at (73.2, 22.6)
- added SW2: SW_Push, Button_Switch_THT:SW_PUSH_6mm, F.Cu at (84.8, 22.6)
- added U5: ESP-12E, ESP8266:ESP-12E_SMD, F.Cu at (114.2, 31.1)
- added U6: OPA330xxDBV, Package_TO_SOT_SMD:SOT-23-5, F.Cu at (57.6, 42.4)
- added U7: 74AHC1G66, Package_TO_SOT_SMD:SOT-353_SC-70-5, F.Cu at (85.3, 83.2)
- C1, C2, C3: footprint Capacitor_SMD:C_0805_2012Metric_Pad1.18x1.45mm_HandSolder -> Capacitor_SMD:C_0805_2012Metric
- J1: footprint Connector_USB:USB_Micro-B_GCT_USB3076-30-A -> Connector_USB:USB_Micro-B_Amphenol_10103594-0001LF_Horizontal
- J2: value ENCODER -> PWR; footprint Connector_PinHeader_2.54mm:PinHeader_1x05_P2.54mm_Vertical -> pl_TerminalBlock:WJ127-5.0-2P
- J3: value AIN -> ESP_PROG; footprint pl_TerminalBlock:WJ127-5.0-2P -> Connector_PinHeader_2.54mm:PinHeader_1x06_P2.54mm_Vertical
- J6: value DB9_Male -> DSUB9_Male
- JP1: value EN_TERM -> Jumper_3_Open; footprint Connector_PinHeader_2.54mm:PinHeader_1x02_P2.54mm_Vertical -> Connector_PinHeader_2.54mm:PinHeader_1x03_P2.54mm_Vertical
- R1: value 0 -> 1k; footprint Resistor_SMD:R_0805_2012Metric_Pad1.20x1.40mm_HandSolder -> Resistor_SMD:R_0805_2012Metric
- R10, R11, R12, R13, R5, R7, R8, R9: footprint Resistor_SMD:R_0805_2012Metric_Pad1.20x1.40mm_HandSolder -> Resistor_SMD:R_0805_2012Metric
- R2: value 10k -> 0; footprint Resistor_SMD:R_0805_2012Metric_Pad1.20x1.40mm_HandSolder -> Resistor_SMD:R_0805_2012Metric
- R3: value 100k -> 0; footprint Resistor_SMD:R_0805_2012Metric_Pad1.20x1.40mm_HandSolder -> Resistor_SMD:R_0805_2012Metric
- R4: value 100k -> 10k; footprint Resistor_SMD:R_0805_2012Metric_Pad1.20x1.40mm_HandSolder -> Resistor_SMD:R_0805_2012Metric
- R6: value 0 -> 10k; footprint Resistor_SMD:R_0805_2012Metric_Pad1.20x1.40mm_HandSolder -> Resistor_SMD:R_0805_2012Metric
- U2: value ESP-01v090 -> BL9342; footprint ESP8266:ESP-01 -> Package_TO_SOT_SMD:SOT-23-6
- moved U2 116.7 mm to (64.7, 134.1)
- moved R2 93.6 mm to (127.7, 119.5), turned to 0 degrees
- moved R3 93.1 mm to (127.8, 123.0)
- moved J1 75.7 mm to (106.5, 96.2), turned to 0 degrees
- moved R5 71.9 mm to (148.9, 124.7)
- moved J3 48.7 mm to (96.6, 22.9), turned to 90 degrees
- moved JP1 33.9 mm to (69.2, 83.4)
- moved R4 23.4 mm to (68.5, 78.3), turned to 0 degrees
- moved R1 20.0 mm to (95.1, 39.6), turned to 0 degrees
- moved R11 18.6 mm to (79.5, 46.5), turned to 0 degrees
- moved J5 16.7 mm to (61.5, 24.6), turned to 180 degrees
- moved R6 15.7 mm to (94.2, 29.4), turned to 90 degrees
- moved R13 14.9 mm to (81.8, 83.5), turned to 270 degrees
- moved R10 14.7 mm to (78.7, 43.1), turned to 270 degrees
- moved U3 10.6 mm to (73.5, 44.0), turned to 0 degrees
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Connections:
- J1 pad 1: +5V -> VBUS
- J1 pad 2: USB_DM -> Net-(J1-Pad2)
- J1 pad 3: USB_DP -> Net-(J1-Pad3)
- J1 pad 6: (no net) -> Net-(J1-Pad6)
- J2 pad 1: +3V3 -> Net-(J2-Pad1)
- J2 pad 2: /ENC_SW -> GND
- J3 pad 2: GND -> FTDI_RX
- J5 pad 1: /AOUT -> Net-(J5-Pad1)
- J6 pad 6: Net-(J6-Pad6) -> GND
- J6 pad 9: Net-(J6-Pad9) -> DSUB_VIN
- JP1 pad 1: /CANH -> DSUB_VIN
- R1 pad 1: USART1_RX -> Net-(D1-Pad1)
- R1 pad 2: Net-(R1-Pad2) -> GPIO0
- R13 pad 1: Net-(JP1-Pad2) -> /CANL
- R13 pad 2: /CANL -> Net-(R13-Pad2)
- R2 pad 1: Net-(R2-Pad1) -> USB_DP
- R2 pad 2: +3V3 -> Net-(J1-Pad3)
- R3 pad 1: Net-(J3-Pad1) -> USB_DM
- R3 pad 2: /ADC_IN1 -> Net-(J1-Pad2)
- R4 pad 1: GND -> Net-(D3-Pad2)
- R4 pad 2: /ADC_IN1 -> GND
- R5 pad 1: +3V3 -> Net-(Q2-Pad2)
- R6 pad 1: Net-(R6-Pad1) -> +3V3
- R6 pad 2: USART1_TX -> RESET
- R8 pad 1: GND -> Net-(R7-Pad1)
- R8 pad 2: Net-(R7-Pad1) -> GND
- R9 pad 1: /AOUT -> AOUT1
- U1 pad 14: Net-(U1-Pad14) -> STM_RESET
- U1 pad 17: /I2C_SCL -> Net-(U1-Pad17)
- U1 pad 18: Net-(U1-Pad18) -> +5V
- U1 pad 21: /I2C_SDA -> Net-(U1-Pad21)
- U1 pad 28: /ADC_IN1 -> Net-(U1-Pad28)
- U1 pad 32: /DAC_OUT1 -> /DAC
- U1 pad 34: Net-(U1-Pad34) -> /PB0
- U1 pad 35: /ENC_SW -> Net-(U1-Pad35)
- U1 pad 36: /ENC_A -> PC1
- U1 pad 38: /ENC_B -> PC0
- U1 pad 39: Net-(U1-Pad39) -> STM_CS
- U1 pad 40: Net-(U1-Pad40) -> STM_RDY
- U1 pad 44: USART1_RX -> STM_RX
- U1 pad 46: Net-(U1-Pad46) -> +5VA
- U1 pad 49: Net-(U1-Pad49) -> SCLK
- U1 pad 51: Net-(U1-Pad51) -> MISO
- U1 pad 53: Net-(U1-Pad53) -> MOSI
- U1 pad 6: +5V -> Net-(U1-Pad6)
- U1 pad 67: Net-(U1-Pad67) -> CAN_TERM
- U1 pad 72: USART1_TX -> STM_TX
- U2 pad 1: Net-(R1-Pad2) -> Net-(C6-Pad2)
- U2 pad 3: Net-(R2-Pad1) -> Net-(C8-Pad2)
- U2 pad 4: Net-(U2-Pad4) -> /Vin
- U2 pad 5: Net-(U2-Pad5) -> /Vin
- U3 pad 1: /AOUT -> AOUT1
- U3 pad 3: /DAC_OUT1 -> DAC1
Routing:
- net USART1_TX: track 73.8 -> 0.00 mm, vias 2 -> 0
- net USB_DP: track 68.2 -> 0.00 mm, vias 2 -> 0
- net /DAC_OUT1: track 65.7 -> 0.00 mm
- net USB_DM: track 61.6 -> 0.00 mm, vias 3 -> 0
- net STM_TX: track 0.00 -> 60.7 mm, vias 0 -> 1
- net /I2C_SDA: track 58.3 -> 0.00 mm
- net /DAC: track 0.00 -> 57.3 mm
- net /I2C_SCL: track 50.3 -> 0.00 mm
- net /ADC_IN1: track 42.7 -> 0.00 mm, vias 2 -> 0
- net MOSI: track 0.00 -> 41.8 mm, vias 0 -> 2
- net MISO: track 0.00 -> 38.8 mm, vias 0 -> 2
- net USART1_RX: track 38.0 -> 0.00 mm, vias 2 -> 0
- net SCLK: track 0.00 -> 37.0 mm, vias 0 -> 2
- net Net-(U1-Pad33): track 33.7 -> 0.00 mm
- net DSUB_VIN: track 0.00 -> 33.6 mm
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- removed copper zone on F.Cu, net +3V3
Other:
- board text added: "AOUT SELECT"
- board text added: "AOUT0"
- board text added: "AOUT1"
- board text added: "BOOT0"
- board text added: "DSUB"
- board text added: "TERM"
- board text removed: "CANalog Beta Dirty Quick Prototype Jan 2021"
- board text removed: "ESP-01"

Commit message: layout getting there
Parts:
- moved R5 72.4 mm to (100.3, 71.0)
- moved Q2 70.1 mm to (102.5, 75.5), turned to 180 degrees
- moved D2 69.9 mm to (104.0, 86.3), turned to 270 degrees
- moved R28 63.9 mm to (100.3, 80.0), turned to 270 degrees
- moved R16 60.5 mm to (103.2, 80.0), turned to 90 degrees
- moved R3 56.3 mm to (106.2, 71.0), turned to 270 degrees
- moved R2 54.3 mm to (103.2, 71.0), turned to 270 degrees
- moved R15 49.6 mm to (108.3, 86.3), turned to 90 degrees
- moved D8 9.25 mm to (31.0, 92.1), turned to 180 degrees
- moved D10 9.03 mm to (31.0, 97.0), turned to 180 degrees
- moved D9 8.57 mm to (31.0, 94.5), turned to 180 degrees
- moved R26 5.76 mm to (34.8, 94.5), turned to 180 degrees
- moved C5 5.71 mm to (93.9, 34.4), turned to 180 degrees
- moved D1 4.42 mm to (94.0, 41.6)
- moved R14 4.42 mm to (93.9, 39.4), turned to 180 degrees
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Connections:
- J1 pad 6: Net-(J1-Pad6) -> GND
Routing:
- net STM_RESET: track 4.17 -> 80.2 mm, vias 0 -> 2
- net GPIO0: track 0.00 -> 36.5 mm
- net Net-(J1-Pad3): track 0.00 -> 26.8 mm, vias 0 -> 2
- net Net-(J1-Pad2): track 0.00 -> 26.0 mm, vias 0 -> 2
- net GPIO2: track 0.00 -> 25.8 mm
- net CH_PD: track 0.00 -> 23.5 mm, vias 0 -> 2
- net USB_DP: track 0.00 -> 19.8 mm
- net +5V: track 48.8 -> 67.4 mm
- net +3V3: track 29.2 -> 46.9 mm, vias 0 -> 2
- net USB_DM: track 0.00 -> 16.1 mm
- net Net-(Q2-Pad1): track 0.00 -> 14.0 mm
- net VBUS: track 0.00 -> 11.3 mm
- net Net-(Q2-Pad2): track 0.00 -> 4.27 mm
- net GND: track 25.3 -> 29.5 mm, vias 16 -> 17
- net RESET: track 26.3 -> 29.4 mm
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
Commit message: Update CANalog_nucleo.kicad_pcb
Parts:
- moved L1 104.8 mm to (85.2, 60.4), turned to 90 degrees
- moved D6 102.5 mm to (91.7, 60.4), turned to 180 degrees
- moved C8 101.4 mm to (85.2, 65.5), turned to 90 degrees
- moved R19 100.3 mm to (76.7, 56.5), turned to 180 degrees
- moved C6 99.0 mm to (81.4, 60.4), turned to 90 degrees
- moved R18 91.4 mm to (81.1, 56.5), turned to 180 degrees
- moved C7 89.8 mm to (88.3, 65.5), turned to 270 degrees
- moved D4 89.0 mm to (81.4, 65.5), turned to 270 degrees
- moved C4 88.4 mm to (76.8, 65.4), turned to 270 degrees
- moved U2 74.7 mm to (76.8, 60.4), turned to 270 degrees
- moved D10 32.5 mm to (56.5, 76.8)
- moved R27 32.5 mm to (60.2, 76.8)
- moved D8 31.3 mm to (56.5, 73.9)
- moved R25 31.3 mm to (60.2, 73.9)
- moved D9 29.5 mm to (56.5, 79.8)
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Routing:
- net +3V3: track 46.9 -> 144.1 mm, vias 2 -> 4
- net +5V: track 67.4 -> 129.2 mm, vias 1 -> 5
- net +5VA: track 0.00 -> 23.2 mm
- net /Vin: track 2.59 -> 25.3 mm
- net Net-(C7-Pad1): track 0.00 -> 19.7 mm
- net PC0: track 0.00 -> 19.2 mm
- net PC1: track 0.00 -> 18.7 mm
- net /PB0: track 0.00 -> 18.5 mm
- net Net-(C8-Pad2): track 0.00 -> 18.0 mm
- net GND: track 29.5 -> 47.4 mm, vias 17 -> 23
- net Net-(C6-Pad1): track 0.00 -> 9.01 mm
- net GPIO0: track 36.5 -> 42.9 mm, vias 0 -> 2
- net Net-(C6-Pad2): track 0.00 -> 3.71 mm
- net Net-(D9-Pad1): track 0.00 -> 2.05 mm
- net Net-(D8-Pad1): track 0.00 -> 2.05 mm
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
Commit message: layout done
Parts:
- added G***: LOGO, PL_logo:logo_height_10mm, F.Cu at (65.8, 61.0)
- moved C9 0.35 mm to (62.2, 44.2)
Routing:
- net +5V: track 129.2 -> 134.6 mm
Other:
- board text added: "CANalog Nucleo Prototype Feb 2021"
- board text added: "CS"
- board text added: "FLASH"
- board text added: "MISO"
- board text added: "MOSI"
- board text added: "PB0"
- board text added: "PC0"
- board text added: "PC1"
- board text added: "RDY"
- board text added: "RESET"
- board text added: "RX"
- board text added: "SCLK"
- board text added: "TX"
- board text added: "cRX"
- board text added: "cTX"
- board text removed: "AOUT SELECT"
