File: pcb/CANalog_nucleo.sch (KiCad schematic (older format))
At the start: 2 parts

Commit message: start schema
Parts:
- added BT?: CR2032, symbol Device:Battery_Cell
- added C? (x2): 0.1uF, symbol Device:C
- added C?: 1uF, symbol Device:C
- added J?: DB9_Male, symbol Connector:DB9_Male
- added J?: ENCODER, symbol Connector_Generic:Conn_01x05
- added J?: OLED, symbol Connector_Generic:Conn_01x04
- added J?: AOUT, symbol Connector_Generic:Conn_01x02
- added JP?: EN_TERM, symbol Device:Jumper_NC_Small
- added R?: 1.5k, symbol Device:R
- added R?: R, symbol Device:R
- added R?: 120, symbol Device:R
- added R?: 68k, symbol Device:R
- added R?: 120k, symbol Device:R
- added R?: 12k, symbol Device:R
- added U?: SN65HVD230, Package_SO:SOIC-8_3.9x4.9mm_P1.27mm, symbol Interface_CAN_LIN:SN65HVD230
- added U? (x3): MCP6002-xSN, symbol Amplifier_Operational:MCP6002-xSN
Connections:
- net +5V: now also C?.1, C?.1, U?.8 (V+)
- net CAN_RX: now also U?.4 (R)
- net CAN_TX: now also U?.1 (D)
- net GND: now also BT?.2 (-), C?.1, C?.2, C?.2, J?.1 (Pin_1), J?.2 (Pin_2), J?.3, J?.5 (Pin_5), R?.1, U?.2 (GND), U?.4 (V-)
- net USB_DP: now also R?.2
- net +3V3: now reaches U?.16 (+3V3)
- net +3V3: now also C?.2, J?.1 (Pin_1), J?.2 (Pin_2), R?.1, U?.3 (VCC)
- net I2C_SCL: now reaches U?.17 (PA15)
- net I2C_SCL: now also J?.3 (Pin_3)
- net I2C_SDA: now reaches U?.21 (PB7)
- net I2C_SDA: now also J?.4 (Pin_4)
- net DAC_OUT1: now reaches U?.32 (PA4)
- net DAC_OUT1: now also U?.3 (+)
- net at U?.33 (VBAT): now also BT?.1 (+)
- net ENC_SW: now reaches U?.35 (PC2)
- net ENC_SW: now also J?.2 (Pin_2)
- net ENC_A: now reaches U?.36 (PC1)
- net ENC_A: now also J?.4 (Pin_4)
- net ENC_B: now reaches U?.38 (PC0)
- net ENC_B: now also J?.3 (Pin_3)
- net CAN_RS: now reaches U?.42 (PC6)
- net CAN_RS: now also R?.2
- new net: R?.1, U?.8 (Rs)
- new net: JP?.2, R?.1
- new net: R?.2, R?.2, U?.2 (-)
- new net: R?.1, R?.2
- new net AOUT: J?.1 (Pin_1), R?.1, U?.1
- new net CANH: J?.7, JP?.1, U?.7 (CANH)
- new net CANL: J?.2, R?.2, U?.6 (CANL)
- no-connect marks 2 -> 12
Other:
- note added: "G = 1 + (Rf/Rin)\nG = 5/3.3"
- moved on the sheet: U?

Commit message: schematic done
Parts:
- added J3: AIN, pl_TerminalBlock:WJ127-5.0-2P, symbol Connector_Generic:Conn_01x02
- added R1, R6: 0, Resistor_SMD:R_0805_2012Metric_Pad1.20x1.40mm_HandSolder, symbol Device:R
- added R10, R11: 20k, Resistor_SMD:R_0805_2012Metric_Pad1.20x1.40mm_HandSolder, symbol Device:R
- added R2: 10k, Resistor_SMD:R_0805_2012Metric_Pad1.20x1.40mm_HandSolder, symbol Device:R
- added R3, R4: 100k, Resistor_SMD:R_0805_2012Metric_Pad1.20x1.40mm_HandSolder, symbol Device:R
- added U2: ESP-01v090, ESP8266:ESP-01, symbol ESP8266:ESP-01v090
- BT1: renamed from BT?; footprint (none) -> Battery:BatteryHolder_Keystone_103_1x20mm
- C1, C2, C3: renamed from C?; footprint (none) -> Capacitor_SMD:C_0805_2012Metric_Pad1.18x1.45mm_HandSolder
- J1: renamed from J?; footprint (none) -> Connector_USB:USB_Micro-B_Amphenol_10103594-0001LF_Horizontal
- J2: renamed from J?; footprint (none) -> Connector_PinHeader_2.54mm:PinHeader_1x05_P2.54mm_Vertical
- J4: renamed from J?; footprint (none) -> Connector_PinHeader_2.54mm:PinHeader_1x04_P2.54mm_Vertical
- J5: renamed from J?; footprint (none) -> pl_TerminalBlock:WJ127-5.0-2P
- J6: renamed from J?; footprint (none) -> Connector_Dsub:DSUB-9_Male_Horizontal_P2.77x2.84mm_EdgePinOffset7.70mm_Housed_MountingHolesOffset9.12mm
- JP1: renamed from JP?; footprint (none) -> Connector_PinHeader_2.54mm:PinHeader_1x02_P2.54mm_Vertical
- R12, R13, R5, R7, R8, R9: renamed from R?; footprint (none) -> Resistor_SMD:R_0805_2012Metric_Pad1.20x1.40mm_HandSolder
- U3: renamed from U?; footprint (none) -> Package_SO:SOIC-8_3.9x4.9mm_P1.27mm
- gave numbers to parts that had none: 2
Connections:
- net +3V3: now also R2.2, U2.7 (VCC)
- net +5V: now also R10.1
- net GND: now also J3.2 (Pin_2), R11.2, R4.1, U2.2 (GND)
- net ADC_IN1: now reaches U1.28 (PA0)
- net ADC_IN1: now also R3.2, R4.2
- net USART1_RX: now reaches U1.44 (PC5)
- net USART1_RX: now also R1.1
- net USART1_TX: now reaches U1.72 (PC4)
- net USART1_TX: now also R6.2
- net at U3.5 (+): now also R10.2, R11.1
- net at U3.6 (-): now also U3.7
- new net: R1.2, U2.1 (UTXD)
- new net: R2.1, U2.3 (CH_PD)
- new net: R6.1, U2.8 (URXD)
- new net: J3.1 (Pin_1), R3.1
- no-connect marks 12 -> 58
Other:
- note added: "0.96" OLED Display"
- note added: "Analog Input Voltage Divider"
- note added: "Analog Output Amplifier"
- note added: "CAN Interface"
- note added: "ESP-01 WiFi Interface"
- note added: "Encoder"
- note added: "Nucleo-F302R8 Connector"
- note added: "Op-Amp"
- note added: "USB Port"
- moved on the sheet: BT1, C1, C2, C3, J1, J2, J4, J5, J6, JP1, R12, R13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

Commit message: quickand dirty prototype
Parts:
- U1: footprint Module:ST_Morpho_Connector_144_STLink -> pl_Nucleo:nucleo-f302r8
Changed lines of the file:
@@
 F 0 "U1" H 3300 5375 50  0000 R CNN
 F 1 "NUCLEO64-F302R8" H 3300 5300 50  0000 R CNN
-F 2 "Module:ST_Morpho_Connector_144_STLink" H 4550 1500 50  0001 L CNN
+F 2 "pl_Nucleo:nucleo-f302r8" H 4550 1500 50  0001 L CNN
 F 3 "" H 3100 2000 50  0001 C CNN
 	1    4000 3400
@@
 	6200 850  6200 950
 $Comp
-L power:GND #PWR?
+L power:GND #PWR0102
 U 1 1 60809ED1
 P 6200 1700
-F 0 "#PWR?" H 6200 1450 50  0001 C CNN
+F 0 "#PWR0102" H 6200 1450 50  0001 C CNN
 F 1 "GND" H 6200 1550 50  0000 C CNN
 F 2 "" H 6200 1700 50  0001 C CNN

Commit message: update schematic
Parts:
- removed BT1: CR2032, Battery:BatteryHolder_Keystone_103_1x20mm, symbol Device:Battery_Cell
- removed J2: ENCODER, Connector_PinHeader_2.54mm:PinHeader_1x05_P2.54mm_Vertical, symbol Connector_Generic:Conn_01x05
- removed J3: AIN, pl_TerminalBlock:WJ127-5.0-2P, symbol Connector_Generic:Conn_01x02
- removed J4: OLED, Connector_PinHeader_2.54mm:PinHeader_1x04_P2.54mm_Vertical, symbol Connector_Generic:Conn_01x04
- removed JP1: EN_TERM, Connector_PinHeader_2.54mm:PinHeader_1x02_P2.54mm_Vertical, symbol Device:Jumper_NC_Small
- removed U2: ESP-01v090, ESP8266:ESP-01, symbol ESP8266:ESP-01v090
- added C10: 1uF, Capacitor_SMD:C_0805_2012Metric, symbol Device:C
- added C11, C6, C9: 0.1uF, Capacitor_SMD:C_0805_2012Metric, symbol Device:C
- added C4: 4.7uF, Capacitor_SMD:C_0805_2012Metric, symbol Device:C
- added C5, C7: 10uF, Capacitor_SMD:C_0805_2012Metric, symbol Device:C
- added C8: 33pF, Capacitor_SMD:C_0603_1608Metric, symbol Device:C
- added D1, D10, D8, D9: LED, LED_SMD:LED_0603_1608Metric, symbol Device:LED
- added D2, D4, D6: SS14F, pl_Diode:SMAF, symbol Device:D_Schottky
- added D3: BZV55-C15, pl_Diode:Nexperia_BZV55_SOD80C, symbol Device:D_Zener
- added D5: 1N4148, Diode_THT:D_DO-35_SOD27_P7.62mm_Horizontal, symbol Device:D
- added D7: PESD1CAN-UX, Package_TO_SOT_SMD:SOT-323_SC-70, symbol pl_diode:PESD1CAN-UX
- added J2: PWR, pl_TerminalBlock:WJ127-5.0-2P, symbol Connector_Generic:Conn_01x02
- added J3: ESP_PROG, Connector_PinHeader_2.54mm:PinHeader_1x06_P2.54mm_Vertical, symbol Connector_Generic:Conn_01x06
- added JP1, JP7, JP8: Jumper_3_Open, Connector_PinHeader_2.54mm:PinHeader_1x03_P2.54mm_Vertical, symbol Jumper:Jumper_3_Open
- added JP2: TX_SELECT, Jumper:SolderJumper-3_P1.3mm_Bridged12_RoundedPad1.0x1.5mm, symbol Jumper:SolderJumper_3_Bridged12
- added JP3: RX_SELECT, Jumper:SolderJumper-3_P1.3mm_Bridged12_RoundedPad1.0x1.5mm, symbol Jumper:SolderJumper_3_Bridged12
- added JP4: BOOT0, Connector_PinHeader_2.54mm:PinHeader_1x02_P2.54mm_Vertical, symbol Device:Jumper_NO_Small
- added JP5: RDY_SELECT, Jumper:SolderJumper-3_P1.3mm_Bridged12_RoundedPad1.0x1.5mm, symbol Jumper:SolderJumper_3_Bridged12
- added JP6: CS_SELECT, Jumper:SolderJumper-3_P1.3mm_Bridged12_RoundedPad1.0x1.5mm, symbol Jumper:SolderJumper_3_Bridged12
- added L1: 2.2uH, pl_Inductor:L_3.5mmx3.0mm_SMD, symbol Device:L
- added Q1: DMP3099L-7, Package_TO_SOT_SMD:SOT-23, symbol Device:Q_PMOS_GSD
- added Q2: MMBT2222A, Package_TO_SOT_SMD:SOT-23, symbol Device:Q_NPN_BEC
- added R14, R15, R17, R21: 10k, Resistor_SMD:R_0805_2012Metric, symbol Device:R
- added R16, R28: 20k, Resistor_SMD:R_0805_2012Metric, symbol Device:R
- added R18: 124k, Resistor_SMD:R_0805_2012Metric, symbol Device:R
- added R19: 23.7k, Resistor_SMD:R_0805_2012Metric, symbol Device:R
- added R20, R25, R26, R27: 1k, Resistor_SMD:R_0805_2012Metric, symbol Device:R
- added R22: 12k, Resistor_SMD:R_0805_2012Metric, symbol Device:R
- added R23: 120k, Resistor_SMD:R_0805_2012Metric, symbol Device:R
- added R24: 68k, Resistor_SMD:R_0805_2012Metric, symbol Device:R
- added SW1, SW2: SW_Push, Button_Switch_THT:SW_PUSH_6mm, symbol Switch:SW_Push
- added U2: BL9342, Package_TO_SOT_SMD:SOT-23-6, symbol pl_DCDC:BL9342
- added U5: ESP-12E, ESP8266:ESP-12E_SMD, symbol ESP8266:ESP-12E
- added U6: OPA330xxDBV, Package_TO_SOT_SMD:SOT-23-5, symbol Amplifier_Operational:OPA330xxDBV
- added U7: 74AHC1G66, Package_TO_SOT_SMD:SOT-353_SC-70-5, symbol pl_analog-switch:74AHC1G66
- C1, C2, C3: footprint Capacitor_SMD:C_0805_2012Metric_Pad1.18x1.45mm_HandSolder -> Capacitor_SMD:C_0805_2012Metric
- J6: value DB9_Male -> DSUB9_Male
- R1: value 0 -> 1k; footprint Resistor_SMD:R_0805_2012Metric_Pad1.20x1.40mm_HandSolder -> Resistor_SMD:R_0805_2012Metric
- R10, R11, R12, R13, R5, R7, R8, R9: footprint Resistor_SMD:R_0805_2012Metric_Pad1.20x1.40mm_HandSolder -> Resistor_SMD:R_0805_2012Metric
- R2: value 10k -> 0; footprint Resistor_SMD:R_0805_2012Metric_Pad1.20x1.40mm_HandSolder -> Resistor_SMD:R_0805_2012Metric
- R3: value 100k -> 0; footprint Resistor_SMD:R_0805_2012Metric_Pad1.20x1.40mm_HandSolder -> Resistor_SMD:R_0805_2012Metric
- R4: value 100k -> 10k; footprint Resistor_SMD:R_0805_2012Metric_Pad1.20x1.40mm_HandSolder -> Resistor_SMD:R_0805_2012Metric
- R6: value 0 -> 10k; footprint Resistor_SMD:R_0805_2012Metric_Pad1.20x1.40mm_HandSolder -> Resistor_SMD:R_0805_2012Metric
Connections:
- net +3V3: now also R6.1, C5.1, D1.2 (A), Q2.3 (C), R14.1, R17.1, R20.1, R21.1, U5.8 (VCC); no longer R2.2, R5.1
- net +5V: now also U1.18 (+5V), C10.1, C11.1, C9.1, D2.1 (K), U6.5 (V+), U7.5 (Vcc); no longer J1.1 (VBUS), U1.6 (E5V)
- net CANH: now also D7.2 (K), U7.1 (Y)
- net CANL: now also R13.1, D7.1 (K); no longer R13.2
- net GND: now also J6.6, R4.2, R8.2, C10.2, C11.2, C4.2, C5.2, C7.2, C9.2, D4.2 (A), D7.3 (A), J2.2 (Pin_2), J3.6 (Pin_6), R19.2, R22.2, R25.1, R26.1, R27.1, R28.2, SW1.1, SW2.1, U2.2 (GND), U5.9 (GND), U6.2 (V-), U7.3 (GND); no longer R4.1, R8.1
- net USB_DM: now also R3.1; no longer J1.2 (D-)
- net USB_DP: now also R2.1; no longer J1.3 (D+)
- net STM_RESET: now reaches U1.14 (~RESET)
- net STM_RESET: now also R21.2, U5.14 (GPIO5)
- net at U1.34 (PB0): now also D8.2 (A)
- net +5VA: now reaches U1.46 (U5V)
- net +5VA: now also D6.1 (K)
- net SCLK: now reaches U1.49 (PB13)
- net SCLK: now also U5.5 (GPIO14)
- net MISO: now reaches U1.51 (PB14)
- net MISO: now also U5.6 (GPIO12)
- net MOSI: now reaches U1.53 (PB15)
- net MOSI: now also U5.7 (GPIO13)
- net CS_NEW: now reaches U1.54 (PB12)
- net CS_NEW: now also JP6.1 (A)
- net CS_OLD: now reaches U1.55 (PB6)
- net CS_OLD: now also JP6.3 (B)
- net RDY_NEW: now reaches U1.56 (PB11)
- net RDY_NEW: now also JP5.1 (A)
- net RDY_OLD: now reaches U1.57 (PC7)
- net RDY_OLD: now also JP5.3 (B)
- net at U1.60 (PB2): now also D10.2 (A)
- net at U1.62 (PB1): now also D9.2 (A)
- net at U1.7 (~BOOT0): now also JP4.2
- net GPIO0: now reaches R1.2
- net GPIO0: now also SW1.2, U5.12 (GPIO0)
- net DSUB_VIN: now reaches J6.9
- net DSUB_VIN: now also JP1.1 (A)
- net at R7.1: now also R8.1; no longer R8.2
- removed net ADC_IN1: R3.2, R4.2, U1.28 (PA0)
- net AOUT renamed AOUT1
- net AOUT1: now also JP8.3 (B); no longer J5.1 (Pin_1)
- net DAC_OUT1 renamed DAC
- net DAC: now also JP7.2 (C); no longer U3.3 (+)
- net ENC_A: no longer names the net of U1.36 (PC1)
- net ENC_B: no longer names the net of U1.38 (PC0)
- net ENC_SW: no longer names the net of U1.35 (PC2)
- net I2C_SCL: no longer names the net of U1.17 (PA15)
- net I2C_SDA renamed CAN_TERM
- net CAN_TERM: now also U7.4 (E)
- net USART1_RX: no longer names the net of R1.1
- net USART1_RX: now also D1.1 (K); no longer U1.44 (PC5)
- net USART1_TX renamed RESET
- net RESET: now also SW2.2, U5.1 (REST); no longer U1.72 (PC4)
- new net: J1.2 (D-), R3.2
- new net: J1.3 (D+), R2.2
- new net: Q2.2 (E), R5.1
- new net: R13.2, U7.2 (Z)
- new net: J5.1 (Pin_1), JP8.2 (C)
- new net: JP4.1, R20.2
- new net: Q2.1 (B), R15.2, R16.1
- new net: R16.2, R28.1
- new net: D5.1 (K), J3.3 (Pin_3)
- new net: J2.1 (Pin_1), JP1.3 (B)
- new net: R23.2, R24.2, U6.4 (-)
- new net: C6.2, U2.1 (BST)
- new net: C8.2, R18.2, R19.1, U2.3 (FB)
- new net: C6.1, D4.1 (K), L1.1, U2.6 (SW)
- new net: D3.2 (A), Q1.1 (G), R4.1
- new net: JP1.2 (C), Q1.3 (D)
- new net: C7.1, C8.1, D6.2 (A), L1.2, R18.1
- new net: R22.1, R23.1
- new net: D9.1 (K), R26.2
- new net: D8.1 (K), R25.2
- new net: D10.1 (K), R27.2
- new net AOUT0: JP8.1 (A), R24.1, U6.1
- new net CH_PD: R17.2, U5.3 (CH_PD)
- new net DAC0: JP7.1 (A), U6.3 (+)
- new net DAC1: JP7.3 (B), U3.3 (+)
- new net ESP_RX: JP3.2 (C), U5.15 (RXD)
- new net ESP_TX: JP2.2 (C), U5.16 (TXD)
- new net FTDI_RX: J3.2 (Pin_2), JP2.1 (A)
- new net FTDI_TX: D5.2 (A), JP3.1 (A)
- new net GPIO2: R14.2, U5.11 (GPIO2)
- new net STM_CS: JP6.2 (C), U5.10 (GPIO15)
- new net STM_RDY: JP5.2 (C), U5.13 (GPIO4)
- new net STM_RX: JP2.3 (B), U1.44 (PC5)
- new net STM_TX: JP3.3 (B), U1.72 (PC4)
- new net VBUS: D2.2 (A), J1.1 (VBUS), R15.1
- new net Vin: C4.1, D3.1 (K), Q1.2 (S), U2.4 (EN), U2.5 (VIN)
- no-connect marks 58 -> 57
Other:
- note added: "AOUT Select"
- note added: "Analog Output - General Purpose Op-Amp"
- note added: "Analog Output - Precision Op-Amp"
- note added: "CAN Terminal"
- note added: "ESP Prog Header"
- note added: "ESP UART Select"
- note added: "External Power 5V Regulator"
- note added: "External Power Input and Select"
- note added: "General Purpose Op-Amp - Unused and Bypass"
- note added: "SPI Controll Select"
- note added: "STM32 USB Pullup"
- note added: "WiFi Interface"
- note removed: "0.96" OLED Display"
- note removed: "Analog Input Voltage Divider"
- note removed: "Analog Output Amplifier"
- note removed: "ESP-01 WiFi Interface"
- note removed: "Encoder"
- note removed: "Op-Amp"
- moved on the sheet: C1, C2, C3, J1, J5, J6, R10, R11, R12, R13, R5, R7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

Commit message: start new pcb layout
Parts:
- removed JP5: RDY_SELECT, Jumper:SolderJumper-3_P1.3mm_Bridged12_RoundedPad1.0x1.5mm, symbol Jumper:SolderJumper_3_Bridged12
- removed JP6: CS_SELECT, Jumper:SolderJumper-3_P1.3mm_Bridged12_RoundedPad1.0x1.5mm, symbol Jumper:SolderJumper_3_Bridged12
Connections:
- net CAN_TERM: now also U1.67 (PB5); no longer U1.21 (PB7)
- net STM_CS: now also U1.39 (PC9)
- net STM_RDY: now also U1.40 (PC8)
- net PB0: now reaches D8.2 (A), U1.34 (PB0)
- net PC1: now reaches U1.36 (PC1)
- net PC1: now also D10.2 (A)
- net PC0: now reaches U1.38 (PC0)
- net PC0: now also D9.2 (A)
- net at U1.60 (PB2): no longer D10.2 (A)
- net at U1.62 (PB1): no longer D9.2 (A)
- net CS_NEW: no longer names the net of U1.54 (PB12)
- net CS_OLD: no longer names the net of U1.55 (PB6)
- net RDY_NEW: no longer names the net of U1.56 (PB11)
- net RDY_OLD: no longer names the net of U1.57 (PC7)
- no-connect marks 57 -> 59
Other:
- note removed: "SPI Controll Select"
Changed lines of the file:
@@
 NoConn ~ 9000 5350
 NoConn ~ 9000 5450
-NoConn ~ 9000 5550
 NoConn ~ 9000 6050
 NoConn ~ 8400 6950
@@
 NoConn ~ 6800 6150
 NoConn ~ 6800 6050
-NoConn ~ 6800 5950
-NoConn ~ 6800 5850
 NoConn ~ 6800 5350
 NoConn ~ 6800 4850
@@
 Wire Wire Line
 	6600 3550 6700 3550
-Wire Wire Line
-	9000 5650 9400 5650
-Wire Wire Line
-	9000 6250 9400 6250
-Text Label 9400 6250 0    50   ~ 0
-CS_NEW
-Text Label 9400 5650 0    50   ~ 0
-CS_OLD
-Text Label 6600 5800 2    50   ~ 0
-RDY_OLD
-Text Label 9400 6150 0    50   ~ 0
-RDY_NEW
-Wire Wire Line
-	9000 6150 9400 6150
-Wire Wire Line
-	6800 5750 6700 5750
-Wire Wire Line
-	6700 5750 6700 5800
-Wire Wire Line
-	6700 5800 6600 5800
 $Comp
 L Device:Jumper_NO_Small JP4
@@
 Wire Wire Line
 	16150 3150 16150 3050
-Text GLabel 9350 5750 2    50   Input ~ 0
+Text GLabel 9350 5550 2    50   Input ~ 0
 CAN_TERM
-Wire Wire Line
-	9350 5750 9000 5750
 Text GLabel 14300 2950 0    50   Input ~ 0
 CAN_TERM
@@
 Wire Wire Line
 	5800 1100 5800 950
-Text GLabel 9250 8800 2    50   Input ~ 0
+Text GLabel 6600 5950 0    50   Input ~ 0
 STM_CS
-Text GLabel 9250 8100 2    50   Input ~ 0
-STM_RDY
-$Comp
-L Jumper:SolderJumper_3_Bridged12 JP5
-U 1 1 6087F94F
-P 8900 8100
-F 0 "JP5" H 8800 8000 50  0000 C CNN
-F 1 "RDY_SELECT" H 8900 8210 50  0000 C CNN
-F 2 "Jumper:SolderJumper-3_P1.3mm_Bridged12_RoundedPad1.0x1.5mm" H 8900 8100 50  0001 C CNN
-F 3 "~" H 8900 8100 50  0001 C CNN
-	1    8900 8100
-	0    -1   1    0
-$EndComp
-$Comp
-L Jumper:SolderJumper_3_Bridged12 JP6
-U 1 1 60881304
-P 8900 8800
-F 0 "JP6" H 8800 8700 50  0000 C CNN
-F 1 "CS_SELECT" H 8900 8910 50  0000 C CNN
-F 2 "Jumper:SolderJumper-3_P1.3mm_Bridged12_RoundedPad1.0x1.5mm" H 8900 8800 50  0001 C CNN
-F 3 "~" H 8900 8800 50  0001 C CNN
-	1    8900 8800
-	0    -1   1    0
-$EndComp
-Wire Wire Line
-	9250 8800 9050 8800
-Wire Wire Line
-	9250 8100 9050 8100
-Text Label 8700 7800 2    50   ~ 0
-RDY_NEW
-Wire Wire Line
-	8700 7800 8900 7800
-Wire Wire Line
-	8900 7800 8900 7900
-Text Label 8700 8400 2    50   ~ 0
-RDY_OLD
-Wire Wire Line
-	8700 8400 8900 8400
-Wire Wire Line
-	8900 8400 8900 8300
-Text Label 8700 9100 2    50   ~ 0
-CS_OLD
-Wire Wire Line
-	8700 9100 8900 9100
-Wire Wire Line
-	8900 9100 8900 9000
-Text Label 8700 8500 2    50   ~ 0
-CS_NEW
-Wire Wire Line
-	8700 8500 8900 8500
-Wire Wire Line
-	8900 8500 8900 8600
-Text Notes 8250 7700 0    50   ~ 0
-SPI Controll Select
-Wire Notes Line
-	8250 7700 9800 7700
-Wire Notes Line
-	9800 9150 8250 9150
-Wire Notes Line
-	8250 9150 8250 7600
-Wire Notes Line
-	8250 7600 9800 7600
-Wire Notes Line
-	9800 7600 9800 9150
 NoConn ~ 9000 4950
-NoConn ~ 6800 5050
-NoConn ~ 6800 5150
 NoConn ~ 6800 5250
 NoConn ~ 9000 3450
@@
 $EndComp
 $Comp
+L Device:R R25
+U 1 1 635EBB6A
+P 10600 5050
+F 0 "R25" V 10680 5050 50  0000 C CNN
+F 1 "1k" V 10600 5050 50  0000 C CNN
+F 2 "Resistor_SMD:R_0805_2012Metric" V 10530 5050 50  0001 C CNN
+F 3 "~" H 10600 5050 50  0001 C CNN
+	1    10600 5050
+	0    1    1    0
+$EndComp
+$Comp
+L Device:LED D8
+U 1 1 635F6452
+P 10200 5050
+F 0 "D8" H 10200 5150 50  0000 C CNN
+F 1 "LED" H 10200 4950 50  0000 C CNN
+F 2 "LED_SMD:LED_0603_1608Metric" H 10200 5050 50  0001 C CNN
+F 3 "~" H 10200 5050 50  0001 C CNN
+	1    10200 5050
+	-1   0    0    1
+$EndComp
+$Comp
+L Device:LED D10
+U 1 1 635F6B4D
+P 10200 5650
+F 0 "D10" H 10200 5750 50  0000 C CNN
+F 1 "LED" H 10200 5550 50  0000 C CNN
+F 2 "LED_SMD:LED_0603_1608Metric" H 10200 5650 50  0001 C CNN
+F 3 "~" H 10200 5650 50  0001 C CNN
+	1    10200 5650
+	-1   0    0    1
+$EndComp
+$Comp
+L Device:R R27
+U 1 1 63627AF7
+P 10600 5650
+F 0 "R27" V 10680 5650 50  0000 C CNN
+F 1 "1k" V 10600 5650 50  0000 C CNN
+F 2 "Resistor_SMD:R_0805_2012Metric" V 10530 5650 50  0001 C CNN
+F 3 "~" H 10600 5650 50  0001 C CNN
+	1    10600 5650
+	0    1    1    0
+$EndComp
+$Comp
+L power:GND #PWR050
+U 1 1 63628CEC
+P 10950 5850
+F 0 "#PWR050" H 10950 5600 50  0001 C CNN
+F 1 "GND" H 10950 5700 50  0000 C CNN
+F 2 "" H 10950 5850 50  0001 C CNN
+F 3 "" H 10950 5850 50  0001 C CNN
+	1    10950 5850
+	1    0    0    -1
+$EndComp
+Wire Wire Line
+	10750 5050 10950 5050
+Wire Wire Line
+	10750 5650 10950 5650
+Wire Wire Line
+	10950 5650 10950 5850
+Wire Wire Line
+	10450 5050 10350 5050
+Wire Wire Line
+	10450 5650 10350 5650
+Wire Wire Line
+	10050 5050 9000 5050
+$Comp
+L Device:R R28
+U 1 1 63887C0E
+P 2650 3700
+F 0 "R28" V 2730 3700 50  0000 C CNN
+F 1 "20k" V 2650 3700 50  0000 C CNN
+F 2 "Resistor_SMD:R_0805_2012Metric" V 2580 3700 50  0001 C CNN
+F 3 "~" H 2650 3700 50  0001 C CNN
+	1    2650 3700
+	1    0    0    -1
+$EndComp
+Wire Wire Line
+	2650 3550 2650 3500
+Text GLabel 6600 5850 0    50   Input ~ 0
+STM_RDY
+Wire Wire Line
+	6600 5850 6800 5850
+NoConn ~ 6800 5750
+Wire Wire Line
+	6600 5950 6800 5950
+NoConn ~ 9000 5650
+NoConn ~ 9000 6150
+NoConn ~ 9000 6250
+Wire Wire Line
+	9000 5550 9350 5550
+NoConn ~ 9000 5750
+Wire Wire Line
+	10450 5350 10350 5350
+Wire Wire Line
+	10750 5350 10950 5350
+$Comp
+L Device:R R26
+U 1 1 636274C8
+P 10600 5350
+F 0 "R26" V 10680 5350 50  0000 C CNN
+F 1 "1k" V 10600 5350 50  0000 C CNN
+F 2 "Resistor_SMD:R_0805_2012Metric" V 10530 5350 50  0001 C CNN
+F 3 "~" H 10600 5350 50  0001 C CNN
+	1    10600 5350
+	0    1    1    0
+$EndComp
+$Comp
 L Device:LED D9
 U 1 1 635E736D
@@
 	-1   0    0    1
 $EndComp
-$Comp
-L Device:R R25
-U 1 1 635EBB6A
-P 10600 5050
-F 0 "R25" V 10680 5050 50  0000 C CNN
-F 1 "1k" V 10600 5050 50  0000 C CNN
-F 2 "Resistor_SMD:R_0805_2012Metric" V 10530 5050 50  0001 C CNN
-F 3 "~" H 10600 5050 50  0001 C CNN
-	1    10600 5050
-	0    1    1    0
-$EndComp
-$Comp
-L Device:LED D8
-U 1 1 635F6452
-P 10200 5050
-F 0 "D8" H 10200 5150 50  0000 C CNN
-F 1 "LED" H 10200 4950 50  0000 C CNN
-F 2 "LED_SMD:LED_0603_1608Metric" H 10200 5050 50  0001 C CNN
-F 3 "~" H 10200 5050 50  0001 C CNN
-	1    10200 5050
-	-1   0    0    1
-$EndComp
-$Comp
-L Device:LED D10
-U 1 1 635F6B4D
-P 10200 5650
-F 0 "D10" H 10200 5750 50  0000 C CNN
-F 1 "LED" H 10200 5550 50  0000 C CNN
-F 2 "LED_SMD:LED_0603_1608Metric" H 10200 5650 50  0001 C CNN
-F 3 "~" H 10200 5650 50  0001 C CNN
-	1    10200 5650
-	-1   0    0    1
-$EndComp
-$Comp
-L Device:R R26
-U 1 1 636274C8
-P 10600 5350
-F 0 "R26" V 10680 5350 50  0000 C CNN
-F 1 "1k" V 10600 5350 50  0000 C CNN
-F 2 "Resistor_SMD:R_0805_2012Metric" V 10530 5350 50  0001 C CNN
-F 3 "~" H 10600 5350 50  0001 C CNN
-	1    10600 5350
-	0    1    1    0
-$EndComp
-$Comp
-L Device:R R27
-U 1 1 63627AF7
-P 10600 5650
-F 0 "R27" V 10680 5650 50  0000 C CNN
-F 1 "1k" V 10600 5650 50  0000 C CNN
-F 2 "Resistor_SMD:R_0805_2012Metric" V 10530 5650 50  0001 C CNN
-F 3 "~" H 10600 5650 50  0001 C CNN
-	1    10600 5650
-	0    1    1    0
-$EndComp
-$Comp
-L power:GND #PWR050
-U 1 1 63628CEC
-P 10950 5850
-F 0 "#PWR050" H 10950 5600 50  0001 C CNN
-F 1 "GND" H 10950 5700 50  0000 C CNN
-F 2 "" H 10950 5850 50  0001 C CNN
-F 3 "" H 10950 5850 50  0001 C CNN
-	1    10950 5850
-	1    0    0    -1
-$EndComp
-Wire Wire Line
-	10750 5050 10950 5050
 Wire Wire Line
 	10950 5050 10950 5350
-Wire Wire Line
-	10750 5650 10950 5650
 Connection ~ 10950 5650
-Wire Wire Line
-	10950 5650 10950 5850
-Wire Wire Line
-	10750 5350 10950 5350
 Connection ~ 10950 5350
 Wire Wire Line
 	10950 5350 10950 5650
-Wire Wire Line
-	10450 5050 10350 5050
-Wire Wire Line
-	10450 5350 10350 5350
-Wire Wire Line
-	10450 5650 10350 5650
-Wire Wire Line
-	10050 5050 9000 5050
-Wire Wire Line
-	9000 5150 10000 5150
+Text Label 9400 5050 2    50   ~ 0
+PB0
+Text GLabel 6600 5050 0    50   Input ~ 0
+PC0
+Text GLabel 6600 5150 0    50   Input ~ 0
+PC1
+Wire Wire Line
+	6600 5050 6800 5050
+Wire Wire Line
+	6600 5150 6800 5150
+Text GLabel 9400 5150 0    50   Input ~ 0
+PC0
+Text GLabel 9400 5250 0    50   Input ~ 0
+PC1
+Wire Wire Line
+	9400 5150 10000 5150
 Wire Wire Line
 	10000 5150 10000 5350
@@
 	9900 5650 9900 5250
 Wire Wire Line
-	9900 5250 9000 5250
-$Comp
-L Device:R R28
-U 1 1 63887C0E
-P 2650 3700
-F 0 "R28" V 2730 3700 50  0000 C CNN
-F 1 "20k" V 2650 3700 50  0000 C CNN
-F 2 "Resistor_SMD:R_0805_2012Metric" V 2580 3700 50  0001 C CNN
-F 3 "~" H 2650 3700 50  0001 C CNN
-	1    2650 3700
-	1    0    0    -1
-$EndComp
-Wire Wire Line
-	2650 3550 2650 3500
+	9900 5250 9400 5250
+NoConn ~ 9000 5150
+NoConn ~ 9000 5250
 $EndSCHEMATC

Commit message: layout getting there
Connections:
- net GND: now also J1.6 (Shield)
- no-connect marks 59 -> 58
Changed lines of the file:
@@
 $EndComp
 Wire Wire Line
-	900  3350 900  3250
+	900  3350 900  3300
 $Comp
 L power:GND #PWR05
@@
 NoConn ~ 6800 4850
 NoConn ~ 13650 1500
-NoConn ~ 800  3250
 $Comp
 L power:PWR_FLAG #FLG0102
@@
 NoConn ~ 9000 5150
 NoConn ~ 9000 5250
+Wire Wire Line
+	800  3250 800  3300
+Wire Wire Line
+	800  3300 900  3300
+Connection ~ 900  3300
+Wire Wire Line
+	900  3300 900  3250
 $EndSCHEMATC
