File: pcb/CANalog.sch (KiCad schematic (older format))
At the start: 89 parts, among them J1 PWR, J2 USB_B_Micro, J3 SPI3, J4 I2C2, J5 STM_PROG, J6 ESP_PROG, J7 AOUT, J8 CAN, Q1 DMP3099L-7, Q2 MMBT2222A, Q3 DMP3099L-7, SW1 SW_Push, SW2 SW_Push, U1 BL9342, U2 LMV321, U3 STM32F302C8T6, U4 MIC5504-3.3YM5, U5 ESP-12E, U6 OPA330xxDBV, U7 74AHC1G66, U8 SN65HVD230, Y1 16MHz

Commit message: add more field info
Parts:
- added JP?: PSELECT, symbol Jumper:Jumper_3_Bridged12
- added R27, R28, R29: 1k, Resistor_SMD:R_0603_1608Metric, symbol Device:R
- C1: MPN (none) -> CL21A475KBQNNNE; Manufacture (none) -> Samsung Electro-Mechanics; SPN (none) -> C98192; Supplier (none) -> LCSC; Supplier Link (none) -> https://lcsc.com/product-detail/Multilayer-Ceramic-Capacito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
- C10, C11, C12, C16, C18, C19, C3, C4, C5, C6, C8: MPN (none) -> C0603C104Z3VACTU; Manufacture (none) -> KEMET; SPN (none) -> 399-1100-1-ND; Supplier (none) -> DigiKey; Supplier Link (none) -> https://www.digikey.com/en/products/detail/kemet/C0603C104Z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
- C13, C15, C17, C2: MPN (none) -> CL10A105KQ8NNNC; Manufacture (none) -> Samsung Electro-Mechanics; SPN (none) -> 1276-1036-1-ND; Supplier (none) -> DigiKey; Supplier Link (none) -> https://www.digikey.com/en/products/detail/samsung-electro-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
- C14, C7: MPN (none) -> CL21A106KPFNNNE; Manufacture (none) -> Samsung Electro-Mechanics; SPN (none) -> C17024; Supplier (none) -> LCSC; Supplier Link (none) -> https://lcsc.com/product-detail/Multilayer-Ceramic-Capacito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
- C9: MPN (none) -> HGC0603G0330J500NTHJ; Manufacture (none) -> Chinocera; SPN (none) -> C465159; Supplier (none) -> LCSC; Supplier Link (none) -> https://lcsc.com/product-detail/Multilayer-Ceramic-Capacito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
- D1: MPN (none) -> BZV55-C15,115; Manufacture (none) -> Nexperia USA Inc.; SPN (none) -> 1727-4962-1-ND; Supplier (none) -> DigiKey; Supplier Link (none) -> https://www.digikey.com/en/products/detail/nexperia-usa-inc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
- D2, D4: Manufacture Shandong Jingdao Microelectronics -> Shandong Jingdao Microelectronics
- D3: value LED -> BLU; MPN (none) -> ORH-B36G; Manufacture (none) -> Orient; SPN (none) -> C193191; Supplier (none) -> LCSC; Supplier Link (none) -> https://lcsc.com/product-detail/Light-Emitting-Diodes-LED_O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
- D6: value LED -> GRN; MPN (none) -> ORH-G36G; Manufacture (none) -> Orient; SPN (none) -> C205443; Supplier (none) -> LCSC; Supplier Link (none) -> https://lcsc.com/product-detail/Light-Emitting-Diodes-LED_O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
- D7: value LED -> ORG; MPN (none) -> NCD0603O1; Manufacture (none) -> Foshan NationStar Optoelectronics; SPN (none) -> C84269; Supplier (none) -> LCSC; Supplier Link (none) -> https://lcsc.com/product-detail/Light-Emitting-Diodes-LED_F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
- D8: value LED -> RED; MPN (none) -> NCD0603R1; Manufacture (none) -> Foshan NationStar Optoelectronics; SPN (none) -> C84263; Supplier (none) -> LCSC; Supplier Link (none) -> https://lcsc.com/product-detail/Light-Emitting-Diodes-LED_F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
- FB1, FB2: Manufacture FH(Guangdong Fenghua Advanced Tech) -> FH(Guangdong Fenghua Advanced Tech)
- J1, J7: MPN (none) -> WJ127-5.0-2P; Manufacture (none) -> Ningbo Kangnex Elec; SPN (none) -> C3703; Supplier (none) -> LCSC; Supplier Link (none) -> https://lcsc.com/product-detail/Screw-terminal_Ningbo-Kangn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
- J2: footprint (none) -> Connector_USB:USB_Micro-B_Molex-105017-0001; MPN (none) -> U254-051T-4BHJ25-S2S; Manufacture (none) -> XKB Connectivity; SPN (none) -> C319163; Supplier (none) -> LCSC; Supplier Link (none) -> https://lcsc.com/product-detail/USB-Connectors_XKB-Connecti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
- J8: MPN (none) -> WJ127-5.0-3P; Manufacture (none) -> Ningbo Kangnex Elec; SPN (none) -> C8393; Supplier (none) -> LCSC; Supplier Link (none) -> https://lcsc.com/product-detail/Screw-terminal_Ningbo-Kangn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
- JP1, JP2: footprint (none) -> Jumper:SolderJumper-2_P1.3mm_Bridged_RoundedPad1.0x1.5mm; Population (none) -> DNP
- L1: MPN (none) -> PSPCAQ32-2R2M; Manufacture (none) -> PROD Tech; SPN (none) -> C436276; Supplier (none) -> LCSC; Supplier Link (none) -> https://lcsc.com/product-detail/Power-Inductors_PROD-Tech-P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
- Q1, Q3: MPN (none) -> DMP3099L-7; Manufacture (none) -> Diodes Incorporated; SPN (none) -> DMP3099L-7DICT-ND; Supplier (none) -> DigiKey; Supplier Link (none) -> https://www.digikey.com/en/products/detail/diodes-incorpora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
- Q2: MPN (none) -> MMBT2222A; Manufacture (none) -> JSMSEMI; SPN (none) -> C916372; Supplier (none) -> LCSC; Supplier Link (none) -> https://lcsc.com/product-detail/Transistors-NPN-PNP_JSMSEMI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
- R11, R22, R23, R24, R8: MPN (none) -> RC0603JR-071KL; Manufacture (none) -> YAGEO; SPN (none) -> 311-1.0KGRCT-ND; Supplier (none) -> DigiKey; Supplier Link (none) -> https://www.digikey.com/en/products/detail/yageo/RC0603JR-0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
- SW1: value SW_Push -> ESP_PROG; footprint (none) -> Button_Switch_SMD:SW_SPST_CK_RS282G05A3; MPN (none) -> TS3625A; Manufacture (none) -> SHOU HAN; SPN (none) -> C398053; Supplier (none) -> LCSC; Supplier Link (none) -> https://lcsc.com/product-detail/Tactile-Switches_SHOU-HAN-T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
- SW2: value SW_Push -> RESET; footprint (none) -> Button_Switch_SMD:SW_SPST_CK_RS282G05A3; MPN (none) -> TS3625A; Manufacture (none) -> SHOU HAN; SPN (none) -> C398053; Supplier (none) -> LCSC; Supplier Link (none) -> https://lcsc.com/product-detail/Tactile-Switches_SHOU-HAN-T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
- TP1: footprint (none) -> TestPoint:TestPoint_Pad_D1.0mm
- U1: MPN (none) -> BL9342; Manufacture (none) -> BL(Shanghai Belling); SPN (none) -> C93176; Supplier (none) -> LCSC; Supplier Link (none) -> https://lcsc.com/product-detail/DC-DC-Converters_BL-Shangha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
- U2: value LMV321 -> RS321BXF; footprint (none) -> Package_TO_SOT_SMD:SOT-23-5; MPN (none) -> RS321BXF; Manufacture (none) -> Jiangsu RUNIC Tech; SPN (none) -> C237022; Supplier (none) -> LCSC; Supplier Link (none) -> https://lcsc.com/product-detail/General-Purpose-Amplifiers_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
- U4: MPN (none) -> MIC5504-3.3YM5-TR; Manufacture (none) -> Microchip Technology; SPN (none) -> 576-4764-1-ND; Supplier (none) -> DigiKey; Supplier Link (none) -> https://www.digikey.com/en/products/detail/MIC5504-3.3YM5-T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
- U5: value ESP-12E -> ESP-12F; MPN (none) -> ESP-12F(ESP8266MOD); Manufacture (none) -> Ai-Thinker; SPN (none) -> C82891; Supplier (none) -> LCSC; Supplier Link (none) -> https://lcsc.com/product-detail/WIFI-Modules_Ai-Thinker-ESP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
Connections:
- net +3V3: now also JP?.1 (A); no longer C18.2, U8.3 (VCC)
- net +5V: now also C19.2, JP?.3 (B); no longer C19.1
- net CANH: now also D10.1 (K), R26.1; no longer D10.2 (K), U7.1 (Y)
- net CANL: now also D10.2 (K), U7.1 (Y); no longer D10.1 (K), R26.1
- net GND: now also C19.1, R27.1, R28.1, R29.1; no longer C19.2
- net V_B0: now reaches U3.18 (PB0)
- net V_B0: now also R29.2
- net V_B1: now reaches U3.19 (PB1)
- net V_B1: now also R28.2
- net V_B2: now reaches U3.20 (PB2)
- net V_B2: now also R27.2
- new net: C18.2, JP?.2 (C), U8.3 (VCC)
Other:
- note added: "0"
- note added: "1"
- note added: "2"
- note added: "3"
- note added: "4"
- note added: "5"
- note added: "6"
- note added: "7"
- note added: "CAN Interface HW Version Indicator"
- note added: "ERC Happy Area"
- note added: "GPIO Internal Pullup"
- note added: "H"
- note added: "L"
- note added: "Mechanical"
- note added: "Reset Circuitry"
- note added: "STM 12bit DAC"
- note added: "STM32F302 IO is 5V tolerent on CAN_TX and CAN_RX GPIO.\nVoltage Selector added to evauate lower cost 5V xcever ICs"
- note added: "This may be used in the future to \nindicate the presence of a 16bit \nDAC or 4 channel output DAC.\nAlso other minor PCB mods as \nrequred. Table will indicate \nversion features when they have \nbeen implemented."
- note added: "V_B0"
- note added: "V_B1"
- note added: "V_B2"
- note added: "Version"
- note removed: "CAN Termination Selection"
- moved on the sheet: C10, C11, C13, C14, C15, C16, C17, C18, C19, C2, C3, C5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
