File: pcb/CANalog.kicad_pcb (KiCad board)
At the start: 2 copper layers, 80 x 45 mm, 82 parts, among them J1 PWR, J4 STM_PROG, J5 ESP_PROG, J6 AOUT, J7 CAN, Q1 DMP3099L-7, SW1 RESET, SW2 ESP_PROG, U1 BL9342, U2 MIC5504-3.3YM5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

Commit message: Update CANalog.kicad_pcb
Parts:
- moved C4 14.4 mm to (67.8, 161.7)
- moved C6 14.4 mm to (62.8, 170.6)
- moved JP1 14.4 mm to (74.6, 174.5)
- moved C10 14.4 mm to (77.5, 167.4)
- moved C2 14.4 mm to (77.5, 173.4)
- moved C8 14.4 mm to (71.8, 175.6)
- moved FB1 14.4 mm to (77.5, 165.4)
- moved R13 14.4 mm to (77.5, 171.4)
- moved R14 14.4 mm to (77.5, 169.4)
- moved U3 14.4 mm to (69.8, 168.7)
- moved Y1 14.4 mm to (80.7, 170.4)
- moved C12 10.0 mm to (102.7, 191.5)
- moved C16 10.0 mm to (84.3, 154.9)
- moved C17 10.0 mm to (84.3, 156.9)
- moved H3 10.0 mm to (92.0, 182.0)
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Routing:
- net +3V3: track 25.5 -> 105.9 mm
- net GPIO0: track 0.00 -> 37.8 mm, vias 0 -> 2
- net ESP_RESET: track 10.4 -> 34.2 mm, vias 0 -> 2
- net STM_RESET: track 22.0 -> 43.4 mm
- net GND: track 21.4 -> 40.6 mm, vias 21 -> 35
- net GPIO2: track 0.00 -> 18.2 mm
- net STM_CS: track 0.00 -> 9.99 mm
- net +BATT: track 0.00 -> 5.85 mm
- net VDDA: track 0.00 -> 5.41 mm
- net GNDA: track 0.00 -> 4.79 mm
- net /XIN: track 0.00 -> 3.98 mm
- net Net-(D7-Pad1): track 0.00 -> 3.03 mm
- net Net-(D9-Pad1): track 0.00 -> 3.02 mm
- net Net-(D8-Pad1): track 0.00 -> 3.02 mm
- net Net-(D10-Pad1): track 0.00 -> 3.02 mm
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Other:
- board size 80 x 45 mm -> 70 x 45 mm

Commit message: update pcb layout, first draft
Parts:
- removed JP1: NC, Jumper:SolderJumper-2_P1.3mm_Bridged_RoundedPad1.0x1.5mm
- NT1: moved to F.Cu
- R21: value R -> 0
- TP1: value PA3 -> PA15
- moved R11 31.0 mm to (75.0, 144.8)
- moved R12 29.9 mm to (75.0, 142.8)
- moved TP1 26.1 mm to (71.6, 177.1)
- moved R16 25.6 mm to (85.0, 177.2)
- moved R10 24.7 mm to (75.0, 146.8)
- moved D4 23.8 mm to (33.3, 158.1)
- moved C12 21.2 mm to (87.8, 176.5), turned to 270 degrees
- moved R8 19.0 mm to (80.7, 180.8), turned to 270 degrees
- moved JP2 16.9 mm to (78.0, 182.1), turned to 180 degrees
- moved J4 12.8 mm to (65.6, 176.6), turned to 0 degrees
- moved NT1 12.2 mm to (77.8, 169.8)
- moved SW1 10.8 mm to (47.5, 181.4)
- moved C8 9.89 mm to (81.5, 177.2), turned to 0 degrees
- moved R18 8.45 mm to (87.1, 156.5), turned to 270 degrees
- moved C2 7.77 mm to (85.0, 175.2)
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Connections:
- C2 pad 1: +BATT -> +3V3
- R21 pad 2: CAN_RS -> GND
- TP1 pad 1: /PA3 -> Net-(TP1-Pad1)
- U3 pad 1: +BATT -> +3V3
- U3 pad 10: CAN_LED -> Net-(U3-Pad10)
- U3 pad 11: SPI_LED -> Net-(U3-Pad11)
- U3 pad 12: ERROR_LED -> Net-(U3-Pad12)
- U3 pad 13: /PA3 -> Net-(U3-Pad13)
- U3 pad 22: STM_RDY -> Net-(U3-Pad22)
- U3 pad 25: STM_CS -> STM_RDY
- U3 pad 29: Net-(U3-Pad29) -> STM_CS
- U3 pad 31: Net-(U3-Pad31) -> CAN_TERM
- U3 pad 32: USB_DM -> CAN_RX
- U3 pad 33: USB_DP -> CAN_TX
- U3 pad 38: Net-(U3-Pad38) -> Net-(TP1-Pad1)
- U3 pad 39: Net-(U3-Pad39) -> CAN_LED
- U3 pad 40: Net-(U3-Pad40) -> SPI_LED
- U3 pad 41: Net-(U3-Pad41) -> ERROR_LED
- U3 pad 42: CAN_RS -> Net-(U3-Pad42)
- U3 pad 43: CAN_TERM -> Net-(U3-Pad43)
- U3 pad 45: CAN_RX -> Net-(U3-Pad45)
- U3 pad 46: CAN_TX -> Net-(U3-Pad46)
Routing:
- net +5V: track 16.5 -> 72.0 mm
- net STM_RDY: track 0.00 -> 45.2 mm, vias 0 -> 2
- net STM_RESET: track 43.4 -> 88.3 mm, vias 0 -> 6
- net STM_CS: track 9.99 -> 52.1 mm, vias 0 -> 4
- net SCLK: track 0.00 -> 35.8 mm, vias 0 -> 2
- net MISO: track 0.00 -> 33.6 mm, vias 0 -> 2
- net MOSI: track 0.00 -> 31.4 mm, vias 0 -> 2
- net CAN_TERM: track 0.00 -> 27.6 mm, vias 0 -> 2
- net V_B0: track 0.00 -> 24.1 mm
- net V_B1: track 0.00 -> 21.9 mm
- net V_B2: track 0.00 -> 19.7 mm
- net CAN_LED: track 0.00 -> 18.6 mm
- net CAN_TX: track 0.00 -> 18.3 mm, vias 0 -> 2
- net +3V3: track 105.9 -> 122.7 mm
- net DAC: track 0.00 -> 15.7 mm
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- added copper zone on B.Cu, net GNDA
- added copper zone on F.Cu, net GNDA

Commit message: clean up and silkscreen work
Parts:
- added G***: LOGO, PL_logo:logo_height_5mm, F.Cu at (92.0, 147.1)
- moved J4 3.92 mm to (61.8, 175.8)
- moved C12 3.89 mm to (85.0, 179.2), turned to 0 degrees
- moved Y1 2.74 mm to (90.8, 173.2)
- moved R18 2.11 mm to (87.7, 158.5)
- moved R20 2.05 mm to (84.9, 158.5)
- moved C17 2.03 mm to (89.9, 153.8)
- moved C16 2.03 mm to (87.4, 153.8)
- moved R19 2.03 mm to (82.1, 158.5)
- moved U5 2.03 mm to (83.2, 153.9)
- moved R26 1.94 mm to (72.0, 152.5)
- moved C18 1.94 mm to (60.6, 152.5)
- moved JP3 1.94 mm to (60.6, 157.3)
- moved C15 1.93 mm to (73.3, 159.9)
- moved U6 1.93 mm to (68.2, 158.7)
- moved U7 1.93 mm to (64.0, 152.6)
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Routing:
- net CAN_TERM: track 27.6 -> 33.2 mm
- net Net-(C9-Pad2): track 5.30 -> 10.8 mm
- net /SWCLK: track 8.97 -> 13.6 mm, vias 0 -> 2
- net +5V: track 72.0 -> 76.4 mm
- net /SWDIO: track 10.3 -> 13.9 mm
- net Net-(R13-Pad2): track 2.51 -> 5.75 mm
- net Net-(R14-Pad2): track 2.51 -> 5.31 mm
- net GND: track 47.9 -> 45.4 mm, vias 41 -> 42
- net Net-(J6-Pad1): track 14.8 -> 17.1 mm
- net DAC: track 15.7 -> 13.7 mm
- net Net-(R18-Pad2): track 5.60 -> 7.43 mm
- net V_B2: track 19.7 -> 18.0 mm
- net +3V3: track 122.7 -> 121.5 mm
- net CAN_TX: track 18.3 -> 17.2 mm
- net GNDA: track 3.74 -> 2.71 mm, vias 47 -> 53
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- removed copper zone on F.Cu, net Net-(C9-Pad2)
Other:
- board text added: "9-30V"
- board text added: "AOUT"
- board text added: "BOOT"
- board text added: "CAN"
- board text added: "CAN_H"
- board text added: "CAN_L"
- board text added: "CANalog"
- board text added: "ERROR"
- board text added: "ESP_PROG"
- board text added: "GND"
- board text added: "GNDA"
- board text added: "May 2021"
- board text added: "RESET"
- board text added: "RX"
- board text added: "SPI"
- board text added: "SWCLK"
- board text added: "SWDIO"
- board text added: "TX"
- board text added: "WIFI"

Commit message: add canalog logo
Parts:
- added G***: LOGO, pl_art:pl_canalog, B.Cu at (48.1, 180.6)

Commit message: cleanup pcb
Parts:
- NT1: moved to B.Cu
Routing:
- net GNDA: track 2.71 -> 5.12 mm
- net GND: track 45.4 -> 47.3 mm, vias 42 -> 41

Commit message: final cleanup
Other:
- board text added: "SSID: CANalog 192.168.1.1"
- board text added: "canalog.io"
